Commit message: update

File: rov_onboard/urdf/rov.urdf.xacro (robot description, xacro)
@@ -2,69 +2,40 @@
 <robot xmlns:xacro="http://www.ros.org/wiki/xacro" name="rov">
 <xacro:property name="PI" value="3.1415926"/>
+  <!-- Left-Bottom of 8020 bar on the ground -->
   <link name="base_link"/>
-    <link name="ahrs_nom"/>
-      <link name="ahrs"/>
-    <link name="left_camera_nom"/>
-      <link name="left_camera"/>
-    <link name="right_camera_nom"/>
-      <link name="right_camera"/>
-    <link name="dvl_nom"/>
-      <link name="dvl"/>
-    <link name="servo_init_nom"/>
-      <link name="servo_init"/>
+    <link name="ahrs"/>
+    <link name="left_camera"/>
+    <link name="right_camera"/>
+    <link name="dvl"/>
+    <link name="sonar"/>
   <!-- ahrs -->
-  <joint name="base_to_ahrs_nom" type="fixed">
+  <joint name="base_to_ahrs" type="fixed">
     <parent link="base_link"/>
-    <child link="ahrs_nom"/>
-    <origin xyz="0.0 0.0 -0.0" rpy="0 0 0"/>
+    <child link="ahrs"/>
+    <origin xyz="0.406 -0.262 0.089" rpy="0 -${PI} 0"/>
   </joint>
-  <joint name="ahrs_nom_to_ahrs" type="fixed">
-    <parent link="ahrs_nom"/>
-    <child link="ahrs"/>
-    <origin xyz="0.0 -0.075 -0.295" rpy="0 0 ${PI/2}"/>
-  </joint>
-  <!-- left camera -->
-  <joint name="base_to_left_camera_nom" type="fixed">
+  <!-- left cam -->
+  <joint name="base_to_left_cam" type="fixed">
     <parent link="base_link"/>
-    <child link="left_camera_nom"/>
+    <child link="left_camera"/>
     <origin xyz="0.0 0.0 0.0" rpy="0 0 0"/>
   </joint>
-  <joint name="left_camera_nom_to_left_camera" type="fixed">
-    <parent link="left_camera_nom"/>
-    <child link="left_camera"/>
-    <origin xyz="-0.28 0.04 -0.1" rpy="${PI} ${-PI/2} 0"/>
-  </joint>
-  <!-- right camera -->
-  <joint name="base_to_right_camera_nom" type="fixed">
+  <!-- right cam -->
+  <joint name="base_to_right_cam" type="fixed">
     <parent link="base_link"/>
-    <child link="right_camera_nom"/>
+    <child link="right_camera"/>
     <origin xyz="0.0 0.0 0.0" rpy="0 0 0"/>
   </joint>
-  <joint name="right_camera_nom_to_right_camera" type="fixed">
-    <parent link="right_camera_nom"/>
-    <child link="right_camera"/>
-    <origin xyz="-0.28 -0.04 -0.1" rpy="${PI} ${-PI/2} 0"/>
+  <!-- dvl -->
+  <joint name="base_to_dvl" type="fixed">
+    <parent link="base_link"/>
+    <child link="dvl"/>
+    <origin xyz="-0.038 -0.159 0.019" rpy="-${PI} 0 0"/>
   </joint>
-  <!-- dvl -->
-  <joint name="base_to_dvl_nom" type="fixed">
+  <!-- sonar -->
+  <joint name="base_to_sonar" type="fixed">
     <parent link="base_link"/>
-    <child link="dvl_nom"/>
-    <origin xyz="0.0 0.0 -0.0" rpy="0 0 0"/>
-  </joint>
-  <joint name="dvl_nom_to_dvl" type="fixed">
-    <parent link="dvl_nom"/>
-    <child link="dvl"/>
-    <origin xyz="-0.45 0.0 0.01" rpy="0 0 0"/>
-  </joint>
-  <!-- servo init -->
-  <joint name="base_to_servo_init_nom" type="fixed">
-    <parent link="base_link"/>
-    <child link="servo_init_nom"/>
-    <origin xyz="0.0 0.0 -0.0" rpy="0 0 0"/>
-  </joint>
-  <joint name="servo_init_nom_to_servo_init" type="fixed">
-    <parent link="servo_init_nom"/>
-    <child link="servo_init"/>
-    <origin xyz="0.28 0.08 -0.3" rpy="0 ${-PI/3} 0"/>
+    <child link="sonar"/>
+    <origin xyz="0.0 0.0 0.0" rpy="0 0 0"/>
   </joint>
 </robot>
