Commit message: update

File: rov_onboard/urdf/rov.urdf (robot description, URDF)
Before this commit: robot rov, 6 links, 5 joints
Links:
- removed link ahrs
- added link microstrain_ahrs
Joints:
- joint base_to_ahrs: child ahrs -> microstrain_ahrs

File: rov_onboard/urdf/rov.urdf.xacro (robot description, xacro)
@@ -4,5 +4,5 @@
   <!-- Left-Bottom of 8020 bar on the ground -->
   <link name="base_link"/>
-    <link name="ahrs"/>
+    <link name="microstrain_ahrs"/>
     <link name="left_camera"/>
     <link name="right_camera"/>
@@ -12,5 +12,5 @@
   <joint name="base_to_ahrs" type="fixed">
     <parent link="base_link"/>
-    <child link="ahrs"/>
+    <child link="microstrain_ahrs"/>
     <origin xyz="0.406 -0.262 0.089" rpy="0 -${PI} 0"/>
   </joint>

File: rov_onboard/urdf/test.urdf (robot description, URDF)
Before this commit: robot rov, 6 links, 5 joints
Links:
- removed link ahrs
- removed link dvl
- added link microstrain_ahrs
- added link nortek_dvl
Joints:
- joint base_to_ahrs: child ahrs -> microstrain_ahrs
- joint base_to_dvl: child dvl -> nortek_dvl
