Commit message: update

File: rov_onboard/urdf/alaska.urdf (robot description, URDF)
Before this commit: robot rov, 6 links, 5 joints
Links:
- removed link dvl
- added link nortek_dvl
Joints:
- joint base_to_dvl: child dvl -> nortek_dvl; origin xyz=-0.038 -0.159 0.019 rpy=-3.1415926 0 0 -> xyz=-0.0635 -0.155575 0.409575 rpy=0 0 0

File: rov_onboard/urdf/rov.urdf.xacro (robot description, xacro)
@@ -7,5 +7,5 @@
     <link name="left_camera"/>
     <link name="right_camera"/>
-    <link name="dvl"/>
+    <link name="nortek_dvl"/>
     <link name="sonar"/>
   <!-- ahrs -->
@@ -30,6 +30,6 @@
   <joint name="base_to_dvl" type="fixed">
     <parent link="base_link"/>
-    <child link="dvl"/>
-    <origin xyz="-0.038 -0.159 0.019" rpy="-${PI} 0 0"/>
+    <child link="nortek_dvl"/>
+    <origin xyz="-0.0635 -0.155575 0.409575" rpy="0 0 0"/>
   </joint>
   <!-- sonar -->

Commit message: update rov_onboard

File: rov_onboard/urdf/alaska.urdf (robot description, URDF)
Before this commit: robot rov, 6 links, 5 joints
Joints:
- joint base_to_sonar: origin xyz=0.0 0.0 0.0 rpy=0 0 0 -> xyz=0.7086 -0.1778 0.2387 rpy=0 -0.2617 0

File: rov_onboard/urdf/rov.urdf (robot description, URDF)
Before this commit: robot rov, 6 links, 5 joints
Joints:
- joint base_to_sonar: origin xyz=0.0 0.0 0.0 rpy=0 0 0 -> xyz=0.7086 -0.1778 0.2387 rpy=0 -0.2617 0

File: rov_onboard/urdf/rov.urdf.xacro (robot description, xacro)
@@ -37,5 +37,5 @@
     <parent link="base_link"/>
     <child link="sonar"/>
-    <origin xyz="0.0 0.0 0.0" rpy="0 0 0"/>
+    <origin xyz="0.7086 -0.1778 0.2387" rpy="0 -0.2617 0"/>
   </joint>
 </robot>
